File: inverter.kicad_pcb (KiCad board)
At the start: 2 copper layers, 45.3 x 22.4 mm, 23 parts, among them P1 CONN_01X02, P2 CONN_01X02, P3 CONN_01X02, U1 LM25576MH

Commit message: Fertig gestellt
Parts:
- added C12: Cout, Capacitors_Tantalum_SMD:TantalC_SizeB_EIA-3528_Reflow, F.Cu at (159.5, 92.6)
- C5: footprint Capacitors_ThroughHole:C_Radial_D6.3_L11.2_P2.5 -> Capacitors_Tantalum_SMD:TantalC_SizeB_EIA-3528_Reflow
- moved C5 10.7 mm to (155.7, 92.6), turned to 90 degrees
- moved C6 9.41 mm to (162.7, 93.3), turned to 270 degrees
Routing:
- net GND: track 48.9 -> 71.4 mm, vias 9 -> 10
- net GNDPWR: track 45.7 -> 27.3 mm, vias 12 -> 9
